File: eagle/ThermoEagle.brd (EAGLE design)
At the start: 100 x 80 mm, 35 parts, among them IC1 MAX232, IC2 4511N, Q1 20MHz, T1 2N2219, T2 2N2219, U1 LM324

Commit message: Temporary update for PCB
Parts:
- moved R1 19.4 mm to (92.7, 10.2)
- moved C8 17.3 mm to (20.3, 71.1), turned to 90 degrees
- moved C3 13.7 mm to (92.7, 73.7), turned to 180 degrees
- moved JP1 13.1 mm to (8.89, 61.0)
- moved C2 12.7 mm to (82.5, 73.7)
- moved J4 11.7 mm to (45.7, 62.2), turned to 270 degrees
- moved R14 9.67 mm to (29.2, 62.2)
- moved C1 8.98 mm to (92.7, 64.8)
- moved C5 8.89 mm to (82.5, 64.8)
- moved C7 6.48 mm to (38.1, 30.5), turned to 270 degrees
- moved T2 6.35 mm to (8.89, 52.1)
- moved J7 5.08 mm to (73.7, 68.6)
- moved R3 5.08 mm to (21.6, 5.08)
- moved S2 4.02 mm to (31.8, 72.4), turned to 270 degrees
- moved J2 3.81 mm to (48.3, 74.9)
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Routing:
- net N$27: track 188.9 -> 55.6 mm
- net N$38: track 183.2 -> 51.1 mm
- net N$70: track 74.2 -> 4.07 mm
- net N$28: track 60.6 -> 124.0 mm
- net VCC: track 341.2 -> 296.9 mm
- net N$4: track 82.8 -> 47.4 mm
- net N$45: track 54.9 -> 88.0 mm
- net N$19: track 6.35 -> 31.1 mm
- net N$31: track 76.7 -> 100.5 mm
- net N$48: track 5.61 -> 28.1 mm
- net N$65: track 4.31 -> 23.5 mm
- net N$17: track 6.88 -> 18.5 mm
- net N$6: track 36.2 -> 46.0 mm
- net N$23: track 20.5 -> 11.0 mm
- net N$7: track 28.2 -> 19.2 mm
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
Commit message: Fix brd file
It's now accepted by EuroCircuit and the teacher launched the print
order.
Routing:
- net N$8: track 0.00 -> 120.4 mm, vias 0 -> 1
- net N$18: track 0.00 -> 3.24 mm, vias 0 -> 1
- net N$5: track 0.00 -> 3.18 mm, vias 0 -> 1
- net GND: track 0.00 -> 2.54 mm, vias 0 -> 1
Changed lines of the file:
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@@
 <setting verticaltext="up"/>
 </settings>
-<grid distance="50" unitdist="mil" unit="mil" style="lines" multiple="1" display="no" altdistance="5" altunitdist="mil" altunit="mil"/>
+<grid distance="25" unitdist="mil" unit="mil" style="lines" multiple="1" display="no" altdistance="5" altunitdist="mil" altunit="mil"/>
 <layers>
 <layer number="1" name="Top" color="4" fill="1" visible="yes" active="yes"/>
@@
 <vertex x="0" y="0"/>
 </polygon>
-<wire x1="29.4894" y1="69.1388" x2="29.4894" y2="75.6412" width="0" layer="19" extent="1-1"/>
+<via x="31.75" y="5.08" extent="1-16" drill="0.35"/>
+<wire x1="34.29" y1="5.08" x2="31.75" y2="5.08" width="0.1524" layer="16"/>
+<wire x1="29.4894" y1="75.6412" x2="29.4894" y2="69.1388" width="0" layer="19" extent="1-1"/>
 <wire x1="34.29" y1="5.08" x2="41.91" y2="15.24" width="0" layer="19" extent="1-1"/>
 </signal>
@@
 <wire x1="34.29" y1="68.961" x2="34.0106" y2="69.1388" width="0.1524" layer="16"/>
 </signal>
+<signal name="N$8">
+<via x="36.83" y="2.54" extent="1-16" drill="0.35"/>
+<wire x1="36.83" y1="2.54" x2="35.56" y2="2.54" width="0.1524" layer="16"/>
+<wire x1="35.56" y1="2.54" x2="34.29" y2="1.27" width="0.1524" layer="16"/>
+<wire x1="34.29" y1="1.27" x2="19.05" y2="1.27" width="0.1524" layer="16"/>
+<wire x1="19.05" y1="1.27" x2="15.875" y2="4.445" width="0.1524" layer="16"/>
+<wire x1="15.875" y1="4.445" x2="1.905" y2="4.445" width="0.1524" layer="16"/>
+<wire x1="1.905" y1="4.445" x2="1.905" y2="48.895" width="0.1524" layer="16"/>
+<wire x1="1.905" y1="48.895" x2="3.81" y2="50.8" width="0.1524" layer="16"/>
+<wire x1="3.81" y1="50.8" x2="3.81" y2="71.12" width="0.1524" layer="16"/>
+<wire x1="3.81" y1="71.12" x2="3.175" y2="71.755" width="0.1524" layer="16"/>
+<wire x1="3.175" y1="71.755" x2="3.175" y2="76.835" width="0.1524" layer="16"/>
+<wire x1="3.175" y1="76.835" x2="10.16" y2="76.835" width="0.1524" layer="16"/>
+<wire x1="10.16" y1="76.835" x2="10.16" y2="73.66" width="0.1524" layer="16"/>
+</signal>
+<signal name="N$5">
+<via x="31.75" y="67.31" extent="1-16" drill="0.35"/>
+<wire x1="29.21" y1="69.215" x2="31.75" y2="67.31" width="0.1524" layer="16"/>
+</signal>
+<signal name="N$18">
+<via x="26.67" y="76.2" extent="1-16" drill="0.35"/>
+<wire x1="26.67" y1="76.2" x2="29.845" y2="75.565" width="0.1524" layer="16"/>
+</signal>
 </signals>
